Commit message: Rosbot description (remove large binary)

File: src/Rosbot_description/urdf/Rosbot.xacro (robot description, xacro)
@@ -88,5 +88,5 @@
   <parent link="base_link"/>
   <child link="left_wheel_1"/>
-  <axis xyz="0.0 -1.0 0.0"/>
+  <axis xyz="0.0 1.0 0.0"/>
 </joint>
 <joint name="right_wheel_joint" type="continuous">
