Commit message: arm controller and arm harware interface added

File: src/noxbot_description_description/urdf/materials.xacro (robot description, xacro)
@@ -4,3 +4,14 @@
   <color rgba="0.700 0.700 0.700 1.000"/>
 </material>
+<material name="blue">
+  <color rgba="0 0 0.5 1" /></material>
+<material name="grey">
+  <color rgba="0.5 0.5 0.5 1" />
+</material>
+<material name="orange">
+  <color rgba="1.0 0.5 0 1" />
+</material>
+<material name="yellow">
+  <color rgba="1.0 1.0 0 1" />
+</material>
 </robot>

File: src/noxbot_description_description/urdf/noxbot_description.xacro (robot description, xacro)
@@ -4,4 +4,7 @@
 <xacro:include filename="$(find noxbot_description_description)/urdf/noxbot_description.ros2control" />
 <xacro:include filename="$(find noxbot_description_description)/urdf/noxbot_description.gazebo" />
+<xacro:include filename="$(find noxbot_description_description)/urdf/arm.xacro" />
+<xacro:property name="base_length" value="0.12" />
+<xacro:property name="base_height" value="0.035" />
 <link name="base_link">
   <inertial>
@@ -130,4 +133,9 @@
   <axis xyz="0 1 0"/>
 </joint>
+<joint name="mobile_base_arm_joint" type="fixed">
+        <parent link="base_link" />
+        <child link="arm_base_link" />
+        <origin xyz="${base_length / 4.0} 0 ${base_height}" rpy="0 0 0" />
+</joint>
 <joint name="front_left_base_joint" type="continuous">
   <origin xyz="0.04726 0.047 0.034" rpy="0 0 0"/>
