Commit message: updated for gz sim

File: src/noxbot_description_description/urdf/arm.xacro (robot description, xacro)
@@ -16,4 +16,15 @@
             <material name="orange" />
         </visual>
+        <collision>
+            <geometry>
+                <box size="${arm_base_length} ${arm_base_width} ${arm_base_height}" />
+            </geometry>
+            <origin xyz="0 0 ${arm_base_height / 2.0}" rpy="0 0 0" />
+        </collision>
+        <inertial>
+            <mass value="0.5" />
+            <origin xyz="0 0 ${arm_base_height / 2.0}" rpy="0 0 0" />
+            <inertia ixx="0.001" iyy="0.001" izz="0.001" ixy="0.0" ixz="0.0" iyz="0.0" />
+        </inertial>
     </link>
     <link name="forearm_link">
@@ -25,4 +36,15 @@
             <material name="yellow" />
         </visual>
+        <collision>
+            <geometry>
+                <cylinder radius="${forearm_radius}" length="${forearm_length}" />
+            </geometry>
+            <origin xyz="0 0 ${forearm_length / 2.0}" rpy="0 0 0" />
+        </collision>
+        <inertial>
+            <mass value="0.3" />
+            <origin xyz="0 0 ${forearm_length / 2.0}" rpy="0 0 0" />
+            <inertia ixx="0.001" iyy="0.001" izz="0.0001" ixy="0.0" ixz="0.0" iyz="0.0" />
+        </inertial>
     </link>
     <link name="hand_link">
@@ -34,4 +56,15 @@
             <material name="orange" />
         </visual>
+        <collision>
+            <geometry>
+                <cylinder radius="${hand_radius}" length="${hand_length}" />
+            </geometry>
+            <origin xyz="0 0 ${hand_length / 2.0}" rpy="0 0 0" />
+        </collision>
+        <inertial>
+            <mass value="0.2" />
+            <origin xyz="0 0 ${hand_length / 2.0}" rpy="0 0 0" />
+            <inertia ixx="0.001" iyy="0.001" izz="0.0001" ixy="0.0" ixz="0.0" iyz="0.0" />
+        </inertial>
     </link>
     <joint name="arm_joint1" type="revolute">

File: src/noxbot_description_description/urdf/noxbot_description.xacro (robot description, xacro)
@@ -6,5 +6,5 @@
 <xacro:include filename="$(find noxbot_description_description)/urdf/arm.xacro" />
 <xacro:property name="base_length" value="0.12" />
-<xacro:property name="base_height" value="0.035" />
+<xacro:property name="base_height" value="0.068" />
 <link name="base_link">
   <inertial>
