Commit message: added virtual right_left_wheel to mimic

File: src/noxbot_description_description/urdf/noxbot_description.xacro (robot description, xacro)
@@ -104,4 +104,30 @@
   </collision>
 </link>
+<link name="left_wheel_link">
+  <inertial>
+    <mass value="0.0001"/>
+    <inertia ixx="1e-6" iyy="1e-6" izz="1e-6"
+             ixy="0" ixz="0" iyz="0"/>
+  </inertial>
+</link>
+<link name="right_wheel_link">
+  <inertial>
+    <mass value="0.0001"/>
+    <inertia ixx="1e-6" iyy="1e-6" izz="1e-6"
+             ixy="0" ixz="0" iyz="0"/>
+  </inertial>
+</link>
+<joint name="left_wheel_joint" type="continuous">
+  <parent link="base_link"/>
+  <child link="left_wheel_link"/>
+  <origin xyz="0.0 0.047 0.034"/>
+  <axis xyz="0 1 0"/>
+</joint>
+<joint name="right_wheel_joint" type="continuous">
+  <parent link="base_link"/>
+  <child link="right_wheel_link"/>
+  <origin xyz="0.0 -0.047 0.034"/>
+  <axis xyz="0 1 0"/>
+</joint>
 <joint name="front_left_base_joint" type="continuous">
   <origin xyz="0.04726 0.047 0.034" rpy="0 0 0"/>
@@ -109,4 +135,5 @@
   <child link="front_left_wheel_1"/>
   <axis xyz="0.0 1.0 0.0"/>
+  <mimic joint="left_wheel_joint"/>
 </joint>
 <joint name="front_right_base_joint" type="continuous">
@@ -115,4 +142,5 @@
   <child link="front_right_wheel_1"/>
   <axis xyz="0.0 1.0 0.0"/>
+  <mimic joint="right_wheel_joint"/>
 </joint>
 <joint name="rear_left_base_joint" type="continuous">
@@ -121,4 +149,5 @@
   <child link="rear_left_wheel_1"/>
   <axis xyz="0.0 1.0 0.0"/>
+  <mimic joint="left_wheel_joint"/>
 </joint>
 <joint name="rear_right_base_joint" type="continuous">
@@ -127,4 +156,5 @@
   <child link="rear_right_wheel_1"/>
   <axis xyz="0.0 1.0 0.0"/>
+  <mimic joint="right_wheel_joint"/>
 </joint>
 </robot>

Commit message: added custom controller

File: src/noxbot_description_description/urdf/noxbot_description.xacro (robot description, xacro)
@@ -6,5 +6,5 @@
 <xacro:include filename="$(find noxbot_description_description)/urdf/arm.xacro" />
 <xacro:property name="base_length" value="0.12" />
-<xacro:property name="base_height" value="0.068" />
+<xacro:property name="base_height" value="0.035" />
 <link name="base_link">
   <inertial>
