Commit message: added bringup with launch file

File: src/noxbot_arm_description/urdf/common_properties.xacro (robot description, xacro)
@@ -8,3 +8,9 @@
     <color rgba="0.0 0.0 0.5 1.0"/>
    </material>
+     <material name="dark_green">
+    <color rgba="0.0 0.4 0.0 1.0"/>
+  </material>
+  <material name="light_green">
+    <color rgba="0.0 0.6 0.0 1.0"/>
+  </material>
 </robot>

File: src/noxbot_arm_description/urdf/noxbot_arm.ros2_control.xacro (robot description, xacro)
@@ -1,7 +1,5 @@
 <?xml version="1.0"?>
 <robot xmlns:xacro="http://www.ros.org/wiki/xacro">
-    <xacro:macro name="noxbot_arm_ros2_control" params="name initial_positions_file">
-        <xacro:property name="initial_positions" value="${load_yaml(initial_positions_file)['initial_positions']}"/>
-        <ros2_control name="${name}" type="system">
+        <ros2_control name="Arm" type="system">
             <hardware>
                 <!-- By default, set up controllers for simulation. This won't work on real hardware -->
@@ -11,5 +9,5 @@
                 <command_interface name="position"/>
                 <state_interface name="position">
-                  <param name="initial_value">${initial_positions['joint1']}</param>
+                  <param name="initial_value">0.0</param>
                 </state_interface>
             </joint>
@@ -17,5 +15,5 @@
                 <command_interface name="position"/>
                 <state_interface name="position">
-                  <param name="initial_value">${initial_positions['joint2']}</param>
+                  <param name="initial_value">0.0</param>
                 </state_interface>
             </joint>
@@ -23,5 +21,5 @@
                 <command_interface name="position"/>
                 <state_interface name="position">
-                  <param name="initial_value">${initial_positions['joint3']}</param>
+                  <param name="initial_value">0.0</param>
                 </state_interface>
             </joint>
@@ -29,5 +27,5 @@
                 <command_interface name="position"/>
                 <state_interface name="position">
-                  <param name="initial_value">${initial_positions['joint4']}</param>
+                  <param name="initial_value">0.0</param>
                 </state_interface>
             </joint>
@@ -35,5 +33,5 @@
                 <command_interface name="position"/>
                 <state_interface name="position">
-                  <param name="initial_value">${initial_positions['joint5']}</param>
+                  <param name="initial_value">0.0</param>
                 </state_interface>
             </joint>
@@ -41,5 +39,5 @@
                 <command_interface name="position"/>
                 <state_interface name="position">
-                  <param name="initial_value">${initial_positions['joint6']}</param>
+                  <param name="initial_value">0.0</param>
                 </state_interface>
             </joint>
@@ -47,8 +45,7 @@
                 <command_interface name="position"/>
                 <state_interface name="position">
-                  <param name="initial_value">${initial_positions['gripper_left_finger_joint']}</param>
+                  <param name="initial_value">0.0</param>
                 </state_interface>
             </joint>
         </ros2_control>
-    </xacro:macro>
 </robot>

File: src/noxbot_arm_description/urdf/noxbot_arm.urdf.xacro (robot description, xacro)
@@ -1,5 +1,12 @@
 <?xml version="1.0"?>
 <robot name="noxbot_arm" xmlns:xacro="http://www.ros.org/wiki/xacro">
-  <xacro:include filename="common_properties.xacro"/>
-  <xacro:include filename="arm.xacro"/>
+  <xacro:include filename="$(find noxbot_arm_description)/urdf/common_properties.xacro"/>
+  <xacro:include filename="$(find noxbot_arm_description)/urdf/arm.xacro"/>
+  <xacro:include filename="$(find noxbot_arm_description)/urdf/gripper.xacro" />
+  <xacro:include filename="$(find noxbot_arm_description)/urdf/noxbot_arm.ros2_control.xacro" />
+  <joint name="gripper_base_joint" type="fixed">
+    <parent link="tool_link"/>
+    <child link="gripper_base_link"/>
+    <origin xyz="0.0 0.0 0.0" rpy="0.0 0.0 0.0"/>
+  </joint>
 </robot>
